Commit message: Initial commit: ROS2 launch file and robot description

File: description/robot.urdf.xacro (robot description, xacro)
@@ -2,3 +2,5 @@
 <robot xmlns:xacro="http://www.ros.org/wiki/xacro"  name="hai_robot">
   <xacro:include filename="robot_core.xacro" />
+  <xacro:include filename="gazebo_control.xacro" />
+  <xacro:include filename="ros2_control.xacro" />
 </robot>

File: description/robot_core.xacro (robot description, xacro)
@@ -34,5 +34,5 @@
         rpy="0 0 0" />
       <geometry>
-        <mesh filename="package://mohd_shan/meshes/base_link.STL"/>
+        <box size="0.3 0.2 0.1"/>
       </geometry>
     </collision>
@@ -71,5 +71,5 @@
         rpy="0 0 0" />
       <geometry>
-        <mesh filename="package://mohd_shan/meshes/Link_BR.STL"/>
+        <cylinder radius="0.033" length="0.03"/>
       </geometry>
     </collision>
@@ -121,5 +121,5 @@
         rpy="0 0 0" />
       <geometry>
-        <mesh filename="package://mohd_shan/meshes/Link_FR.STL"/>
+        <cylinder radius="0.033" length="0.03"/>
       </geometry>
     </collision>
@@ -170,5 +170,5 @@
         rpy="0 0 0" />
       <geometry>
-        <mesh filename="package://mohd_shan/meshes/Link_FL.STL"/>
+        <cylinder radius="0.033" length="0.03"/>
       </geometry>
     </collision>
@@ -219,5 +219,5 @@
         rpy="0 0 0" />
       <geometry>
-        <mesh filename="package://mohd_shan/meshes/Link_BL.STL"/>
+        <cylinder radius="0.033" length="0.03"/>
       </geometry>
     </collision>
