Commit message: Initial commit

File: description/gazebo_control.xacro (robot description, xacro)
@@ -1,6 +1,6 @@
+<?xml version="1.0"?>
 <robot xmlns:xacro="http://www.ros.org/wiki/xacro">
   <gazebo>
-    <plugin name="gz::sim::systems::DiffDrive"
-            filename="gz-sim-diff-drive-system">
+    <plugin name="gz::sim::systems::DiffDrive" filename="gz-sim-diff-drive-system">
       <left_joint>joint_FL</left_joint>
       <left_joint>joint_BL</left_joint>
@@ -9,6 +9,7 @@
       <wheel_separation>0.19</wheel_separation>
       <wheel_radius>0.033</wheel_radius>
-      <topic>cmd_vel</topic>
-      <odom_topic>odom</odom_topic>
+      <topic>/cmd_vel</topic>
+      <odom_topic>/odom</odom_topic>
+      <tf_topic>/model/my_bot/tf</tf_topic>
       <frame_id>odom</frame_id>
       <child_frame_id>base_link</child_frame_id>
@@ -16,9 +17,5 @@
     <plugin name="gz::sim::systems::JointStatePublisher"
             filename="gz-sim-joint-state-publisher-system">
-      <topic>joint_states</topic>
-      <joint_name>joint_FL</joint_name>
-      <joint_name>joint_BL</joint_name>
-      <joint_name>joint_FR</joint_name>
-      <joint_name>joint_BR</joint_name>
+      <topic>/joint_states</topic>
     </plugin>
   </gazebo>

File: description/robot.urdf.xacro (robot description, xacro)
@@ -1,6 +1,6 @@
 <?xml version="1.0"?>
-<robot xmlns:xacro="http://www.ros.org/wiki/xacro"  name="hai_robot">
-  <xacro:include filename="robot_core.xacro" />
-  <xacro:include filename="gazebo_control.xacro" />
-  <xacro:include filename="ros2_control.xacro" />
+<robot name="hai_robot" xmlns:xacro="http://www.ros.org/wiki/xacro">
+  <xacro:include filename="$(find mohd_shan)/description/robot_core.xacro"/>
+  <xacro:include filename="$(find mohd_shan)/description/lidar.xacro"/>
+  <xacro:include filename="$(find mohd_shan)/description/gazebo_control.xacro"/>
 </robot>

File: description/robot_core.xacro (robot description, xacro)
@@ -1,73 +1,38 @@
 <?xml version="1.0"?>
 <robot name="hai_robot" xmlns:xacro="http://www.ros.org/wiki/xacro">
+  <!-- BASE LINK -->
   <link name="base_link">
     <inertial>
-      <origin
-        xyz="0.000368761558726893 0.000222079211190218 -0.0186832943864639"
-        rpy="0 0 0" />
-      <mass
-        value="0.921963005425886" />
-      <inertia
-        ixx="0.00268947436013833"
-        ixy="-8.01568946641351E-06"
-        ixz="8.59504316907562E-07"
-        iyy="0.00489558963627434"
-        iyz="1.75461888359984E-06"
-        izz="0.00732819171596806" />
+      <origin xyz="0 0 0.075" rpy="0 0 0"/>
+      <mass value="8.0"/>
+      <inertia ixx="0.08" iyy="0.12" izz="0.18" ixy="0.0" ixz="0.0" iyz="0.0"/>
     </inertial>
     <visual>
-      <origin
-        xyz="0 0 0"
-        rpy="0 0 0" />
       <geometry>
-        <mesh filename="package://mohd_shan/meshes/base_link.STL"/>
+        <mesh filename="package://mohd_shan/meshes/base_link.stl" scale="0.001 0.001 0.001"/>
       </geometry>
-      <material
-        name="">
-        <color
-          rgba="0.792156862745098 0.819607843137255 0.933333333333333 1" />
-      </material>
     </visual>
     <collision>
-      <origin
-        xyz="0 0 0"
-        rpy="0 0 0" />
+      <origin xyz="0 0 0.075"/>
       <geometry>
-        <box size="0.3 0.2 0.1"/>
+        <box size="0.30 0.20 0.06"/>
       </geometry>
     </collision>
   </link>
-  <link name="Link_BR">
+  <!-- ========= WHEELS ========= -->
+  <!-- FRONT RIGHT -->
+  <link name="Link_FR">
     <inertial>
-      <origin
-        xyz="0 0.0074934 -2.2204E-16"
-        rpy="0 0 0" />
-      <mass
-        value="0.074247" />
-      <inertia
-        ixx="3.0786E-05"
-        ixy="1.9378E-19"
-        ixz="3.8312E-21"
-        iyy="5.884E-05"
-        iyz="-2.0715E-19"
-        izz="3.0786E-05" />
+      <mass value="0.35"/>
+      <inertia ixx="0.001" iyy="0.001" izz="0.001"/>
     </inertial>
     <visual>
-      <origin
-        xyz="0 0 0"
-        rpy="0 0 0" />
+      <origin xyz="-0.095294 0.124382 -0.009657"/>
       <geometry>
-        <mesh filename="package://mohd_shan/meshes/Link_BR.STL"/>
+        <mesh filename="package://mohd_shan/meshes/wheel_FR_1.stl" scale="0.001 0.001 0.001"/>
       </geometry>
-      <material
-        name="">
-        <color
-          rgba="0.79216 0.81961 0.93333 1" />
-      </material>
     </visual>
+    <!-- FIXED: collision aligned -->
     <collision>
-      <origin
-        xyz="0 0 0"
-        rpy="0 0 0" />
       <geometry>
         <cylinder radius="0.033" length="0.03"/>
@@ -75,49 +40,24 @@
     </collision>
   </link>
-  <joint name="joint_BR"
-    type="continuous">
-    <origin
-      xyz="-0.10018 -0.1126 -0.058355"
-      rpy="0 0 0" />
-    <parent
-      link="base_link" />
-    <child
-      link="Link_BR" />
-    <axis
-      xyz="0 1 0" />
+  <joint name="joint_FR" type="continuous">
+    <parent link="base_link"/>
+    <child link="Link_FR"/>
+    <origin xyz="0.095294 -0.124382 0.033"/>
+    <axis xyz="0 -1 0"/>
+    <dynamics damping="1.0" friction="0.2"/>
   </joint>
-  <link
-    name="Link_FR">
+  <!-- FRONT LEFT -->
+  <link name="Link_FL">
     <inertial>
-      <origin
-        xyz="1.1102E-16 0.0074934 -2.2204E-16"
-        rpy="0 0 0" />
-      <mass
-        value="0.074247" />
-      <inertia
-        ixx="3.0786E-05"
-        ixy="1.959E-19"
-        ixz="-6.8527E-34"
-        iyy="5.884E-05"
-        iyz="-9.7951E-20"
-        izz="3.0786E-05" />
+      <mass value="0.35"/>
+      <inertia ixx="0.001" iyy="0.001" izz="0.001"/>
     </inertial>
     <visual>
-      <origin
-        xyz="0 0 0"
-        rpy="0 0 0" />
+      <origin xyz="-0.095294 -0.090848 -0.009657"/>
       <geometry>
-        <mesh filename="package://mohd_shan/meshes/Link_FR.STL"/>
+        <mesh filename="package://mohd_shan/meshes/wheel_FL_1.stl" scale="0.001 0.001 0.001"/>
       </geometry>
-      <material
-        name="">
-        <color
-          rgba="0.79216 0.81961 0.93333 1" />
-      </material>
     </visual>
     <collision>
-      <origin
-        xyz="0 0 0"
-        rpy="0 0 0" />
       <geometry>
         <cylinder radius="0.033" length="0.03"/>
@@ -125,48 +65,24 @@
     </collision>
   </link>
-  <joint name="joint_FR"
-    type="continuous">
-    <origin
-      xyz="0.10018 -0.1126 -0.058355"
-      rpy="0 0 0" />
-    <parent
-      link="base_link" />
-    <child
-      link="Link_FR" />
-    <axis
-      xyz="0 1 0" />
+  <joint name="joint_FL" type="continuous">
+    <parent link="base_link"/>
+    <child link="Link_FL"/>
+    <origin xyz="0.095294 0.090848 0.033"/>
+    <axis xyz="0 -1 0"/>
+    <dynamics damping="1.0" friction="0.2"/>
   </joint>
-  <link name="Link_FL">
+  <!-- BACK LEFT -->
+  <link name="Link_BL">
     <inertial>
-      <origin
-        xyz="1.1102E-16 -0.0074934 0"
-        rpy="0 0 0" />
-      <mass
-        value="0.074247" />
-      <inertia
-        ixx="3.0786E-05"
-        ixy="-3.6573E-20"
-        ixz="-1.3332E-21"
-        iyy="5.884E-05"
-        iyz="2.2518E-19"
-        izz="3.0786E-05" />
+      <mass value="0.35"/>
+      <inertia ixx="0.001" iyy="0.001" izz="0.001"/>
     </inertial>
     <visual>
-      <origin
-        xyz="0 0 0"
-        rpy="0 0 0" />
+      <origin xyz="0.105062 -0.090848 -0.009657"/>
       <geometry>
-        <mesh filename="package://mohd_shan/meshes/Link_FL.STL"/>
+        <mesh filename="package://mohd_shan/meshes/wheel_BL_1.stl" scale="0.001 0.001 0.001"/>
       </geometry>
-      <material
-        name="">
-        <color
-          rgba="0.79216 0.81961 0.93333 1" />
-      </material>
     </visual>
     <collision>
-      <origin
-        xyz="0 0 0"
-        rpy="0 0 0" />
       <geometry>
         <cylinder radius="0.033" length="0.03"/>
@@ -174,48 +90,24 @@
     </collision>
   </link>
-  <joint name="joint_FL"
-    type="continuous">
-    <origin
-      xyz="0.10018 0.1126 -0.058355"
-      rpy="0 0 0" />
-    <parent
-      link="base_link" />
-    <child
-      link="Link_FL" />
-    <axis
-      xyz="0 1 0" />
+  <joint name="joint_BL" type="continuous">
+    <parent link="base_link"/>
+    <child link="Link_BL"/>
+    <origin xyz="-0.105062 0.090848 0.033"/>
+    <axis xyz="0 -1 0"/>
+    <dynamics damping="1.0" friction="0.2"/>
   </joint>
-  <link name="Link_BL">
+  <!-- BACK RIGHT -->
+  <link name="Link_BR">
     <inertial>
-      <origin
-        xyz="-4.4409E-16 -0.0074934 -4.4409E-16"
-        rpy="0 0 0" />
-      <mass
-        value="0.074247" />
-      <inertia
-        ixx="3.0786E-05"
-        ixy="1.3418E-24"
-        ixz="4.0908E-37"
-        iyy="5.884E-05"
-        iyz="-3.0264E-19"
-        izz="3.0786E-05" />
+      <mass value="0.35"/>
+      <inertia ixx="0.001" iyy="0.001" izz="0.001"/>
     </inertial>
     <visual>
-      <origin
-        xyz="0 0 0"
-        rpy="0 0 0" />
+      <origin xyz="0.105062 0.124382 -0.009657"/>
       <geometry>
-        <mesh filename="package://mohd_shan/meshes/Link_BL.STL"/>
+        <mesh filename="package://mohd_shan/meshes/wheel_BR_1.stl" scale="0.001 0.001 0.001"/>
       </geometry>
-      <material
-        name="">
-        <color
-          rgba="0.79216 0.81961 0.93333 1" />
-      </material>
     </visual>
     <collision>
-      <origin
-        xyz="0 0 0"
-        rpy="0 0 0" />
       <geometry>
         <cylinder radius="0.033" length="0.03"/>
@@ -223,15 +115,10 @@
     </collision>
   </link>
-  <joint name="joint_BL"
-    type="continuous">
-    <origin
-      xyz="-0.10018 0.1126 -0.058355"
-      rpy="0 0 0" />
-    <parent
-      link="base_link" />
-    <child
-      link="Link_BL" />
-    <axis
-      xyz="0 1 0" />
+  <joint name="joint_BR" type="continuous">
+    <parent link="base_link"/>
+    <child link="Link_BR"/>
+    <origin xyz="-0.105062 -0.124382 0.033"/>
+    <axis xyz="0 -1 0"/>
+    <dynamics damping="1.0" friction="0.2"/>
   </joint>
 </robot>

File: description/ros2_control.xacro (robot description, xacro)
@@ -1,49 +1,3 @@
-<xacro:if value="$(arg sim_mode)">
-  <ros2_control name="GazeboSystem" type="system">
-    <hardware>
-      <plugin>gz_ros2_control/GazeboSimSystem</plugin>
-    </hardware>
-    <joint name="left_wheel_joint">
-      <command_interface name="velocity"/>
-    </joint>
-    <joint name="left_front_wheel_joint">
-      <command_interface name="velocity">
-        <param name="min">-10</param>
-        <param name="max">10</param>
-      </command_interface>
-      <state_interface name="velocity"/>
-      <state_interface name="position"/>
-    </joint>
-    <joint name="left_rear_wheel_joint">
-      <command_interface name="velocity">
-        <param name="min">-10</param>
-        <param name="max">10</param>
-      </command_interface>
-      <state_interface name="velocity"/>
-      <state_interface name="position"/>
-    </joint>
-    <joint name="right_front_wheel_joint">
-      <command_interface name="velocity">
-        <param name="min">-10</param>
-        <param name="max">10</param>
-      </command_interface>
-      <state_interface name="velocity"/>
-      <state_interface name="position"/>
-    </joint>
-    <joint name="right_rear_wheel_joint">
-      <command_interface name="velocity">
-        <param name="min">-10</param>
-        <param name="max">10</param>
-      </command_interface>
-      <state_interface name="velocity"/>
-      <state_interface name="position"/>
-    </joint>
-  </ros2_control>
-</xacro:if>
-<gazebo>
-  <plugin name="gz_ros2_control::GazeboSimROS2ControlPlugin"
-          filename="libgz_ros2_control-system.so">
-    <parameters>$(find articubot_one)/config/my_controllers.yaml</parameters>
-    <parameters>$(find articubot_one)/config/gaz_ros2_ctl_use_sim.yaml</parameters>
-  </plugin>
-</gazebo>
+<?xml version="1.0"?>
+<robot xmlns:xacro="http://www.ros.org/wiki/xacro">
+</robot>
